Commit message: Renamed sample_vehicle_description package to nissan_leaf_description

File: nissan_leaf_description/urdf/vehicle.xacro (robot description, xacro)
@@ -2,5 +2,5 @@
 <robot xmlns:xacro="http://ros.org/wiki/xacro">
   <!-- load parameter -->
-  <xacro:property name="vehicle_info" value="${load_yaml('$(find sample_vehicle_description)/config/vehicle_info.param.yaml')}"/>
+  <xacro:property name="vehicle_info" value="${load_yaml('$(find nissan_leaf_description)/config/vehicle_info.param.yaml')}"/>
   <!-- vehicle body -->
   <link name="base_link">
@@ -8,5 +8,5 @@
       <origin xyz="${vehicle_info['/**']['ros__parameters']['wheel_base']/2.0} 0 0" rpy="${pi/2.0} 0 ${pi}"/>
       <geometry>
-        <mesh filename="package://sample_vehicle_description/mesh/lexus.dae" scale="1 1 1"/>
+        <mesh filename="package://nissan_leaf_description/mesh/NissanLeafZE0.dae" scale="1 1 1"/>
       </geometry>
     </visual>

Commit message: Adjusted naming and parameters to fit Nissan Leaf

File: nissan_leaf_description/urdf/vehicle.xacro (robot description, xacro)
@@ -6,5 +6,5 @@
   <link name="base_link">
     <visual>
-      <origin xyz="${vehicle_info['/**']['ros__parameters']['wheel_base']/2.0} 0 0" rpy="${pi/2.0} 0 ${pi}"/>
+      <origin xyz="1.08 0 0" rpy="0 0 ${pi/2.0}"/>
       <geometry>
         <mesh filename="package://nissan_leaf_description/mesh/NissanLeafZE0.dae" scale="1 1 1"/>
